File: 7segment.kicad_sch (KiCad schematic)
At the start: 30 parts, among them J1 AVR-ISP-6, J2 Conn_01x10, J4 Conn_01x02, Q1 Q_NPN_BEC, Q2 Q_NPN_BEC, U1 ATmega168PA-AU, U2 HDSP-523

Commit message: Update
Parts:
- U1: symbol MCU_Microchip_ATmega:ATmega168PA-AU -> MCU_Microchip_ATmega:ATmega168PA-A
Connections:
- net +5V renamed VCC
Other:
- title: Hex display for breadboards -> 7 Segment Hex Display

Commit message: Update
Connections:
- net ZERO_I_OR_LE renamed ZERO_I_OR_OE
Other:
- note added: "At 50% duty cycle: Red HDSP-523E 270 ohms Green HDSP-523G 120 ohms Yellow HDSP-523Y 100 ohms"
- note added: "If mode is open: Works with zero blanking chaining. if Pin 1 is high, display both zeros, and drive pin 10 high if Pin 1 is low, zeroes become blank, and if the value is zero on both displays, drive pin 10 low If mode is closed: Pin 1 becomes Output Enable. when low: only the right dot is turned on to signify power when high: display functions normally"
- note removed: "At 50% duty cycle: Red 270 ohms Green 120 ohms Yellow 100 ohms"
- moved on the sheet: C1, C2, C3, C4, C5, C6, D1, J1, J2, J4, JP1, L1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
